File: WBDR_02/WBDR_02.sch (EAGLE design)
At the start: 44 parts, among them IC1 TLP175A_TPL,E, IC2 DIO6970TST6, IC3 SN65HVD232D, IC4 TLP175A_TPL,E, IC5 TLP175A_TPL,E, IC7 DS05-127-2-04BK-SMT-TR

Commit message: HW finished
Parts:
- removed IC7: DS05-127-2-04BK-SMT-TR, SamacSys_Parts:DS05-127-2-04BK-SMT-TR
- renumbered REL1 to RELAY1, REL2 to RELAY2, REL3 to RELAY3
Connections:
- removed net O4: OUTS.2, RELAY3.COM_2, RELAY3.NO_2
- removed net SCL: IC7.COM_2, IC7.COM_4
- removed net SCL1: IC7.NO_2
- removed net SCL2: IC7.NO_4
- removed net SDA: IC7.COM_1, IC7.COM_3
- removed net SDA1: IC7.NO_1
- removed net SDA2: IC7.NO_3
- new net IN1: OUTS.5, RELAY1.COM_2, RELAY1.NO_2
- new net IN2: OUTS.3, RELAY2.COM_2, RELAY2.NO_2
- net +3V3: no longer OUTS.1
- net GND: no longer RELAY1.COM_1
- net O1: now also OUTS.4, RELAY1.COM_1, RELAY1.NO_1; no longer OUTS.5, RELAY1.COM_2
- net O2: now also OUTS.2, RELAY2.COM_1, RELAY2.NO_1; no longer OUTS.4, RELAY1.NO_2
- net O3: now also OUTS.1, RELAY3.COM_2, RELAY3.NO_2; no longer OUTS.3, RELAY2.COM_2, RELAY2.NO_2
- net VIN: no longer RELAY1.NO_1, RELAY2.COM_1, RELAY2.NO_1
