File: WBD_02/WBD_02.brd (EAGLE design)
At the start: 30.9 x 64 mm, 40 parts, among them IC2 DIO6970TST6, IC3 SN65HVD232D, IC4 DS3231M+TRL, IC5 AT24C32D-SSHM-B, IC7 DS05-127-2-04BK-SMT-TR

Commit message: Change CAN and add new board WBDR
Parts:
- removed I2C, UART: (no value), pinhead:1X03
- added JP1: (no value), pinhead:1X06
Connections:
- net +3V3: now also JP1.1
- net CANRX: now also ESP32.15; no longer ESP32.4
- net CANTX: now also ESP32.16; no longer ESP32.5
- net GND: now also JP1.6; no longer I2C.3, UART.3
- net LED2: now also ESP32.28; no longer ESP32.18
- net RX: now also JP1.4; no longer UART.1
- net SCL2: now also JP1.3; no longer I2C.2
- net SDA2: now also JP1.2; no longer I2C.1
- net TX: now also JP1.5; no longer UART.2
Routing:
- net CANRX: track 56.7 -> 37.0 mm, vias 2 -> 0
- net CANTX: track 52.2 -> 33.8 mm, vias 2 -> 0
- net LED2: track 20.1 -> 4.05 mm, vias 2 -> 0
- net +3V3: track 147.7 -> 156.2 mm
- net SDA2: track 18.8 -> 23.0 mm
- net SCL2: track 23.3 -> 27.4 mm

Commit message: HW finished
Parts:
- moved R5 2.42 mm to (28.1, 42.7)
- moved LED 2.42 mm to (28.1, 39.2)
- renumbered JP1 to UART/I2C
Connections:
- removed net MTCK: ESP32.32, MICROSD.5
- removed net MTDI: ESP32.34, MICROSD.7
- removed net MTDO: ESP32.33, MICROSD.3
- new net MISO: ESP32.30, MICROSD.7
- new net MOSI: ESP32.28, MICROSD.3
- new net SCK: ESP32.29, MICROSD.5
- net LED2: now also ESP32.27; no longer ESP32.28
- net SCL: now also ESP32.38, ESP32.5
- net SDA: now also ESP32.39, ESP32.4; no longer ESP32.23
- net SDCARD: now also ESP32.31; no longer ESP32.26
Routing:
- net MOSI: track 0.00 -> 19.2 mm, vias 0 -> 1
- net SCL: track 4.63 -> 23.2 mm, vias 0 -> 1
- net MTDI: track 16.2 -> 0.00 mm, vias 1 -> 0
- net SCK: track 0.00 -> 14.7 mm, vias 0 -> 1
- net MISO: track 0.00 -> 11.9 mm, vias 0 -> 1
- net MTCK: track 11.4 -> 0.00 mm, vias 1 -> 0
- net MTDO: track 11.1 -> 0.00 mm, vias 1 -> 0
- net SDCARD: track 23.6 -> 13.3 mm
- net SDA: track 19.6 -> 23.1 mm
