File: HW/WBD_02_OBD2X/WBD_02_OBD2X.brd (EAGLE design)
At the start: 30.9 x 64 mm, 3 parts

Commit message: Codigo general y expansion OBD2
Parts:
- added OBD2: OBD2, OBD2:OBD2
Connections:
- new net CHASIS: OBD2.4
- net CANH: now also OBD2.6
- net CANL: now also OBD2.14
- net GND: now also OBD2.13, OBD2.5
- net VEXT: now also OBD2.16
Routing:
- net GND: track 0.00 -> 59.2 mm
- net CANH: track 0.00 -> 26.9 mm
- net VEXT: track 0.00 -> 16.3 mm
- net CANL: track 0.00 -> 15.3 mm
- added copper zone on layer 1, net CHASIS
- added copper zone on layer 16, net CHASIS
- removed copper zone on layer 1, net GND
- removed copper zone on layer 16, net GND
Changed lines of the file:
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@@
 <setting verticaltext="up"/>
 </settings>
-<grid distance="5" unitdist="mil" unit="mil" style="lines" multiple="1" display="yes" altdistance="5" altunitdist="mil" altunit="mil"/>
+<grid distance="25" unitdist="mil" unit="mil" style="lines" multiple="1" display="yes" altdistance="5" altunitdist="mil" altunit="mil"/>
 <layers>
 <layer number="1" name="Top" color="4" fill="1" visible="yes" active="yes"/>
@@
 <layer number="14" name="Route14" color="1" fill="6" visible="no" active="no"/>
 <layer number="15" name="Route15" color="4" fill="6" visible="no" active="no"/>
-<layer number="16" name="Bottom" color="1" fill="1" visible="yes" active="yes"/>
+<layer number="16" name="Bottom" color="1" fill="1" visible="no" active="yes"/>
 <layer number="17" name="Pads" color="2" fill="1" visible="yes" active="yes"/>
 <layer number="18" name="Vias" color="2" fill="1" visible="yes" active="yes"/>
@@
 <attribute name="VALUE" x="25.273" y="36.195" size="1.27" layer="27" rot="R270"/>
 </element>
+<element name="OBD2" library="OBD2" package="OBD2" value="OBD2" x="29.464" y="16.129" smashed="yes" rot="R90">
+<attribute name="NAME" x="5.464" y="13.129" size="1.27" layer="21" rot="R90"/>
+</element>
 </elements>
 <signals>
 <signal name="GND">
-<polygon width="0.1524" layer="1" spacing="0.254" isolate="0.254">
-<vertex x="0" y="56.388"/>
-<vertex x="30.988" y="56.388"/>
+<contactref element="VBAT" pad="2"/>
+<contactref element="UART/I2C" pad="6"/>
+<contactref element="OBD2" pad="5"/>
+<contactref element="OBD2" pad="13"/>
+<wire x1="19.464" y1="30.129" x2="21.941" y2="30.129" width="1.016" layer="16"/>
+<wire x1="21.941" y1="30.129" x2="26.035" y2="26.035" width="1.016" layer="16"/>
+<wire x1="26.035" y1="26.035" x2="26.035" y2="23.495" width="1.016" layer="16"/>
+<wire x1="26.035" y1="23.495" x2="27.305" y2="22.225" width="1.016" layer="16"/>
+<wire x1="27.305" y1="22.225" x2="28.448" y2="22.225" width="1.016" layer="16"/>
+<wire x1="10.464" y1="30.129" x2="6.634" y2="30.129" width="1.016" layer="16"/>
+<wire x1="6.634" y1="30.129" x2="5.08" y2="28.575" width="1.016" layer="16"/>
+<wire x1="5.08" y1="28.575" x2="5.08" y2="13.335" width="1.016" layer="16"/>
+<wire x1="7.112" y1="11.303" x2="28.448" y2="11.303" width="1.016" layer="16"/>
+<wire x1="5.08" y1="13.335" x2="7.112" y2="11.303" width="1.016" layer="16"/>
+<wire x1="10.464" y1="30.129" x2="19.464" y2="30.129" width="0" layer="19" extent="1-1"/>
+</signal>
+<signal name="+3V3">
+<contactref element="UART/I2C" pad="1"/>
+</signal>
+<signal name="CANL">
+<contactref element="CAN" pad="2"/>
+<contactref element="OBD2" pad="14"/>
+<wire x1="19.464" y1="26.129" x2="22.766" y2="26.129" width="0.6096" layer="16"/>
+<wire x1="25.781" y1="18.034" x2="28.448" y2="18.034" width="0.6096" layer="16"/>
+<wire x1="22.766" y1="26.129" x2="24.13" y2="24.765" width="0.6096" layer="16"/>
+<wire x1="24.13" y1="19.685" x2="25.781" y2="18.034" width="0.6096" layer="16"/>
+<wire x1="24.13" y1="24.765" x2="24.13" y2="19.685" width="0.6096" layer="16"/>
+</signal>
+<signal name="CANH">
+<contactref element="CAN" pad="1"/>
+<contactref element="OBD2" pad="6"/>
+<wire x1="10.464" y1="26.129" x2="13.876" y2="26.129" width="0.6096" layer="16"/>
+<wire x1="15.24" y1="24.765" x2="15.24" y2="17.145" width="0.6096" layer="16"/>
+<wire x1="16.891" y1="15.494" x2="28.448" y2="15.494" width="0.6096" layer="16"/>
+<wire x1="13.876" y1="26.129" x2="15.24" y2="24.765" width="0.6096" layer="16"/>
+<wire x1="15.24" y1="17.145" x2="16.891" y2="15.494" width="0.6096" layer="16"/>
+</signal>
+<signal name="RX">
+<contactref element="UART/I2C" pad="4"/>
+</signal>
+<signal name="TX">
+<contactref element="UART/I2C" pad="5"/>
+</signal>
+<signal name="VEXT">
+<contactref element="VBAT" pad="1"/>
+<contactref element="OBD2" pad="16"/>
+<wire x1="19.464" y1="18.129" x2="19.464" y2="12.286" width="1.016" layer="1"/>
+<wire x1="22.987" y1="8.763" x2="28.448" y2="8.763" width="1.016" layer="1"/>
+<wire x1="19.464" y1="12.286" x2="22.987" y2="8.763" width="1.016" layer="1"/>
+</signal>
+<signal name="SDA2">
+<contactref element="UART/I2C" pad="2"/>
+</signal>
+<signal name="SCL2">
+<contactref element="UART/I2C" pad="3"/>
+</signal>
+<signal name="CHASIS">
+<contactref element="OBD2" pad="4"/>
+<polygon width="0.1524" layer="16" spacing="0.254" isolate="0.254">
+<vertex x="0" y="64.388"/>
+<vertex x="30.988" y="64.388"/>
 <vertex x="30.988" y="0"/>
 <vertex x="0" y="0"/>
 </polygon>
-<polygon width="0.1524" layer="16" spacing="0.254" isolate="0.254">
-<vertex x="0" y="56.388"/>
-<vertex x="30.988" y="56.388"/>
+<polygon width="0.1524" layer="1" spacing="0.254" isolate="0.254">
+<vertex x="0" y="64.388"/>
+<vertex x="30.988" y="64.388"/>
 <vertex x="30.988" y="0"/>
 <vertex x="0" y="0"/>
 </polygon>
-<contactref element="VBAT" pad="2"/>
-<contactref element="UART/I2C" pad="6"/>
-<wire x1="28.448" y1="11.303" x2="28.448" y2="22.225" width="0" layer="19" extent="1-1"/>
-</signal>
-<signal name="+3V3">
-<contactref element="UART/I2C" pad="1"/>
-</signal>
-<signal name="CANL">
-<contactref element="CAN" pad="2"/>
-</signal>
-<signal name="CANH">
-<contactref element="CAN" pad="1"/>
-</signal>
-<signal name="RX">
-<contactref element="UART/I2C" pad="4"/>
-</signal>
-<signal name="TX">
-<contactref element="UART/I2C" pad="5"/>
-</signal>
-<signal name="VEXT">
-<contactref element="VBAT" pad="1"/>
-</signal>
-<signal name="SDA2">
-<contactref element="UART/I2C" pad="2"/>
-</signal>
-<signal name="SCL2">
-<contactref element="UART/I2C" pad="3"/>
 </signal>
 </signals>
