File: HW/WBD_03/WBD_03.brd (EAGLE design)
At the start: 30.9 x 64 mm, 40 parts, among them IC2 DIO6970TST6, IC3 SN65HVD232D, IC4 DS3231M+TRL, IC5 AT24C32D-SSHM-B, IC7 DS05-127-2-04BK-SMT-TR

Commit message: Finish WBD_03 + gerbers
Routing:
- net USBD-: track 56.8 -> 60.8 mm
- net VIN: track 45.8 -> 48.4 mm, vias 1 -> 4
- net USBD+: track 54.9 -> 57.3 mm, vias 0 -> 2
Other:
- outline, holes or cut-outs redrawn
